Commit message: feat(ur5): transfer the visual of ur5 to primitives

File: tests/data/ur5/ur5_primitive.urdf (robot description, URDF)
Before this commit: robot ur5, 11 links, 10 joints
Links:
- link base_link: geometry collision mesh filename=collision/base.stl; visual cylinder length=0.02 radius=0.075
- link forearm_link: geometry collision mesh filename=collision/forearm.stl; visual cylinder length=0.47 radius=0.035
- link shoulder_link: geometry collision mesh filename=collision/shoulder.stl; visual cylinder length=0.13 radius=0.056
- link upper_arm_link: geometry collision mesh filename=collision/upperarm.stl; visual cylinder length=0.53 radius=0.056
- link wrist_1_link: geometry collision mesh filename=collision/wrist1.stl; visual cylinder length=0.105 radius=0.035
- link wrist_2_link: geometry collision mesh filename=collision/wrist2.stl; visual cylinder length=0.115 radius=0.035
- link wrist_3_link: geometry collision mesh filename=collision/wrist3.stl; visual cylinder length=0.025 radius=0.036
Joints:
- joint shoulder_pan_joint: origin xyz=0.0 0.0 0.089159 rpy=0.0 0.0 0.0 -> xyz=0.0 0.0 0.08 rpy=0.0 0.0 0.0

Commit message: fix(ur5): only collision meshed should be changed to primitives

File: tests/data/ur5/ur5_primitive.urdf (robot description, URDF)
Before this commit: robot ur5, 11 links, 10 joints
Links:
- link base_link: geometry collision cylinder length=0.025 radius=0.075; visual mesh filename=collision/base.stl
- link forearm_link: geometry collision cylinder length=0.47 radius=0.035; visual mesh filename=collision/forearm.stl
- link shoulder_link: geometry collision cylinder length=0.13 radius=0.056; visual mesh filename=collision/shoulder.stl
- link upper_arm_link: geometry collision cylinder length=0.53 radius=0.056; visual mesh filename=collision/upperarm.stl
- link wrist_1_link: geometry collision cylinder length=0.105 radius=0.035; visual mesh filename=collision/wrist1.stl
- link wrist_2_link: geometry collision cylinder length=0.115 radius=0.035; visual mesh filename=collision/wrist2.stl
- link wrist_3_link: geometry collision cylinder length=0.025 radius=0.036; visual mesh filename=collision/wrist3.stl
Joints:
- joint shoulder_pan_joint: origin xyz=0.0 0.0 0.08 rpy=0.0 0.0 0.0 -> xyz=0.0 0.0 0.089159 rpy=0.0 0.0 0.0

Commit message: feat(ur5): enlarge the collision primitive size to avoid collision

File: tests/data/ur5/ur5_primitive.urdf (robot description, URDF)
Before this commit: robot ur5, 11 links, 10 joints
Links:
- link forearm_link: geometry collision cylinder length=0.49 radius=0.045; visual mesh filename=collision/forearm.stl
- link shoulder_link: geometry collision cylinder length=0.13 radius=0.065; visual mesh filename=collision/shoulder.stl
- link upper_arm_link: geometry collision cylinder length=0.53 radius=0.062; visual mesh filename=collision/upperarm.stl
- link wrist_1_link: geometry collision cylinder length=0.105 radius=0.045; visual mesh filename=collision/wrist1.stl
- link wrist_2_link: geometry collision cylinder length=0.11 radius=0.045; visual mesh filename=collision/wrist2.stl
- link wrist_3_link: geometry collision cylinder length=0.03 radius=0.04; visual mesh filename=collision/wrist3.stl

Commit message: fix(ur5_primitive): remove end effector collision since it's not used

File: tests/data/ur5/ur5_primitive.urdf (robot description, URDF)
Before this commit: robot ur5, 11 links, 10 joints
Links:
- link ee_link: geometry 
